File: Macro_Keyboard.kicad_pcb (KiCad board)
At the start: 4 copper layers, 95.6 x 84.2 mm, 115 parts, among them J1 USB_C_Receptacle_USB2.0, J2 USB_A, J3 USB_A, J4 USB_A, SW1 SW_Push, SW10 SW_DIP_x01, SW2 SW_DIP_x01, SW3 SW_DIP_x01, SW4 SW_DIP_x01, SW5 SW_DIP_x01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

Commit message: Add files via upload
Parts:
- moved R14 59.5 mm to (128.0, 81.3), turned to 180 degrees
- moved SK6812MINI_E4 41.9 mm to (76.3, 96.8), turned to 0 degrees
- moved C5 41.6 mm to (145.9, 84.7), turned to 0 degrees
- moved SK6812MINI_E6 35.2 mm to (114.7, 96.8), turned to 0 degrees
- moved C14 26.7 mm to (126.6, 75.9), turned to 90 degrees
- moved C3 21.9 mm to (130.1, 75.5), turned to 90 degrees
- moved C4 19.7 mm to (131.9, 75.5), turned to 90 degrees
- moved U2 16.5 mm to (134.7, 75.4), turned to -90 degrees
- moved R12 13.9 mm to (137.8, 53.0), turned to -90 degrees
- moved C1 13.8 mm to (137.4, 73.5), turned to 90 degrees
- moved C2 12.4 mm to (139.1, 73.5), turned to 90 degrees
- moved C33 10.7 mm to (83.4, 80.3), turned to 180 degrees
- moved C36 10.6 mm to (121.8, 118.4), turned to 180 degrees
- moved C31 10.6 mm to (121.7, 80.4), turned to 180 degrees
- moved C32 10.6 mm to (102.6, 80.4), turned to 180 degrees
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Routing:
- net COL 0: track 0.00 -> 114.3 mm, vias 0 -> 2
- net GND: track 0.00 -> 88.0 mm, vias 0 -> 20
- net COL 1: track 0.00 -> 82.5 mm, vias 0 -> 3
- net +5V: track 0.00 -> 79.4 mm, vias 0 -> 26
- net ROW 2: track 0.00 -> 75.8 mm, vias 0 -> 2
- net ROW 0: track 0.00 -> 74.9 mm, vias 0 -> 2
- net Net-(U1-NRST): track 0.00 -> 71.0 mm, vias 0 -> 1
- net ROW 1: track 0.00 -> 66.2 mm, vias 0 -> 2
- net COL 2: track 0.00 -> 61.4 mm, vias 0 -> 2
- net +3.3V: track 0.00 -> 59.7 mm, vias 0 -> 7
- net Net-(U1-PH3): track 0.00 -> 52.6 mm, vias 0 -> 1
- net Rotary_A: track 0.00 -> 42.2 mm, vias 0 -> 1
- net SDA: track 0.00 -> 41.5 mm
- net Rotary_B: track 0.00 -> 35.4 mm, vias 0 -> 1
- net DVDD: track 0.00 -> 29.8 mm, vias 0 -> 4
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- added copper zone on In2.Cu, net +3.3V
- added copper zone on In2.Cu, net +5V
- added copper zone on In2.Cu, net AVDD
- added copper zone on In2.Cu, net DVDD
- added copper zone on B.Cu, net GND
- added copper zone on F.Cu, net GND
- added copper zone on In1.Cu, net GND
Other:
- board text added: "Orientation from LEDS Note Add !!!"

Commit message: Add files via upload
Parts:
- added ?: , , F.Cu at (67.3, 118.1)
- added ?: , , F.Cu at (152.9, 119.9)
- added ?: , , F.Cu at (67.3, 44.5)
- added ?: , , F.Cu at (151.4, 49.2)
- moved C19 0.10 mm to (149.7, 63.5)
Routing:
- net /USB/D_P3: track 92.4 -> 96.1 mm
- net /USB/D_N3: track 92.3 -> 94.9 mm
- net GND: track 88.0 -> 90.3 mm, vias 20 -> 86
- net /USB/D_P1: track 46.7 -> 47.9 mm
- net /USB/D_N1: track 46.6 -> 47.5 mm
- net Net-(J2-VBUS): track 17.8 -> 18.4 mm
Other:
- board size 95.6 x 84.2 mm -> 95.5 x 83.8 mm
- board text added: "Stundner 2023 Macro Keyboard Rev. 0.7"
- board text removed: "Orientation from LEDS Note Add !!!"

Commit message: Add files via upload
Parts:
- removed ? (x4): , 
- moved SK6812MINI_E6 1.06 mm to (115.8, 96.8)
- moved SK6812MINI_E5 1.06 mm to (96.7, 96.8)
- moved SK6812MINI_E1 1.01 mm to (117.2, 80.7)
- moved SK6812MINI_E7 0.97 mm to (117.2, 118.8)
- moved SK6812MINI_E4 0.97 mm to (77.3, 96.8)
- moved SK6812MINI_E2 0.85 mm to (98.1, 80.7)
- moved SK6812MINI_E8 0.85 mm to (97.9, 118.8)
- moved SK6812MINI_E3 0.85 mm to (78.8, 80.7)
- moved SK6812MINI_E9 0.85 mm to (78.8, 118.8)
Routing:
- net /USB/D_P3: track 96.1 -> 92.5 mm
- net /USB/D_N3: track 94.9 -> 91.4 mm
- net GND: track 90.3 -> 88.4 mm, vias 86 -> 88
- net LED: track 17.3 -> 18.9 mm
- net /USB/D_P2: track 63.3 -> 62.3 mm
- net /USB/D_N2: track 63.2 -> 62.3 mm
- net /USB/D_N1: track 47.5 -> 46.6 mm
- net /USB/D_P1: track 47.9 -> 47.0 mm
- net +5V: track 79.4 -> 78.7 mm
- net DVDD: track 29.8 -> 29.1 mm
- net Net-(U1-NRST): track 71.0 -> 71.6 mm
Other:
- board text added: "Stundner 2023 Macro Keyboard Rev. 0.8"
- board text removed: "Stundner 2023 Macro Keyboard Rev. 0.7"

Commit message: Add files via upload
Parts:
- added H1: MountingHole_Pad, MountingHole:MountingHole_2.2mm_M2_DIN965_Pad, F.Cu at (66.5, 44.7)
- added H2: MountingHole_Pad, MountingHole:MountingHole_2.2mm_M2_DIN965_Pad, F.Cu at (66.0, 119.4)
- added H3: MountingHole_Pad, MountingHole:MountingHole_2.2mm_M2_DIN965_Pad, F.Cu at (153.4, 119.1)
- added H4: MountingHole_Pad, MountingHole:MountingHole_2.2mm_M2_DIN965_Pad, F.Cu at (151.4, 49.3)
- C1: footprint Inductor_SMD:L_0603_1608Metric_Pad1.05x0.95mm_HandSolder -> Capacitor_SMD:C_0603_1608Metric_Pad1.08x0.95mm_HandSolder
- moved C1 4.79 mm to (132.7, 74.4), turned to 180 degrees
- moved C20 3.07 mm to (134.3, 72.3), turned to 0 degrees
- moved Y1 3.05 mm to (137.4, 69.1)
- moved R17 2.80 mm to (150.9, 45.9), turned to 0 degrees
- moved C2 2.76 mm to (136.5, 74.4), turned to 180 degrees
- moved C21 2.61 mm to (140.5, 72.3), turned to 180 degrees
- moved C3 1.78 mm to (130.1, 77.3)
- moved C4 1.78 mm to (131.9, 77.3)
- moved U2 1.78 mm to (134.7, 77.2)
- moved D2 1.52 mm to (150.9, 75.5)
- moved R16 1.52 mm to (150.9, 79.8)
- moved R4 1.52 mm to (150.9, 77.6)
- moved R13 0.49 mm to (150.9, 43.7), turned to 0 degrees
Routing:
- net GND: track 88.4 -> 106.0 mm, vias 88 -> 93
- net +5V: track 78.7 -> 83.4 mm
- net /USB/X1: track 17.0 -> 13.3 mm
- net Net-(J1-CC2): track 13.0 -> 9.32 mm
- net COL 2: track 61.4 -> 59.6 mm
- net /USB/X2: track 13.0 -> 11.2 mm
- net Net-(U1-NRST): track 71.6 -> 73.3 mm
- net Net-(U1-PB3): track 3.61 -> 5.13 mm
- net SDA: track 41.5 -> 42.4 mm
