File: Macro_Keyboard.kicad_pcb (KiCad board)
At the start: 4 copper layers, 95.5 x 83.8 mm, 119 parts, among them J1 USB_C_Receptacle_USB2.0, J2 USB_A, J3 USB_A, J4 USB_A, SW1 SW_Push, SW10 SW_DIP_x01, SW2 SW_DIP_x01, SW3 SW_DIP_x01, SW4 SW_DIP_x01, SW5 SW_DIP_x01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

Commit message: Add files via upload
Parts:
- added C45: 0.1uF, Capacitor_SMD:C_0603_1608Metric_Pad1.08x0.95mm_HandSolder, F.Cu at (154.0, 103.1)
- added C46: 0.1uF, Capacitor_SMD:C_0603_1608Metric_Pad1.08x0.95mm_HandSolder, F.Cu at (152.0, 105.4)
- added R18: 10k, Resistor_SMD:R_0805_2012Metric_Pad1.20x1.40mm_HandSolder, F.Cu at (153.2, 98.5)
- added R19: 10k, Resistor_SMD:R_0805_2012Metric_Pad1.20x1.40mm_HandSolder, F.Cu at (151.1, 98.5)
- added U7: NUP2202, Package_TO_SOT_SMD:TSOT-23-6, F.Cu at (117.9, 58.9)
- added U8: NUP2202, Package_TO_SOT_SMD:TSOT-23-6, F.Cu at (98.8, 59.4)
- U5: value SRV05-4 -> NUP2202; footprint Package_TO_SOT_SMD:SOT-23-6 -> Package_TO_SOT_SMD:TSOT-23-6; moved to B.Cu
- U6: value SRV05-4 -> NUP2202; footprint Package_TO_SOT_SMD:SOT-23-6 -> Package_TO_SOT_SMD:TSOT-23-6
- moved U6 15.8 mm to (79.2, 60.7), turned to 0 degrees
- moved U5 12.0 mm to (141.6, 53.3)
- moved TH1 3.87 mm to (112.6, 61.2)
- moved R2 0.16 mm to (132.1, 112.6), turned to 0 degrees
Connections:
- MT1 pad A: Rotary_A -> Net-(C45-Pad1)
- MT1 pad B: Rotary_B -> Net-(C46-Pad1)
- R2 pad 1: Net-(MT1-Pad2) -> GND
- R2 pad 2: GND -> Net-(MT1-Pad2)
- U5 pad 3: /USB/D_N0 -> unconnected-(U5-Pad3)
- U5 pad 4: /USB/D_N1 -> unconnected-(U5-Pad4)
- U5 pad 6: /USB/D_P1 -> /USB/D_N0
- U6 pad 1: /USB/D_P2 -> /USB/D_P3
- U6 pad 3: /USB/D_N2 -> unconnected-(U6-Pad3)
- U6 pad 4: /USB/D_P3 -> unconnected-(U6-Pad4)
Routing:
- net Rotary_A: track 42.3 -> 21.9 mm
- net /USB/D_P1: track 47.0 -> 26.8 mm, vias 2 -> 0
- net /USB/D_N1: track 46.6 -> 26.3 mm, vias 2 -> 0
- net Net-(C45-Pad1): track 0.00 -> 19.4 mm
- net /USB/D_P3: track 92.5 -> 77.0 mm
- net Rotary_B: track 35.4 -> 20.1 mm
- net /USB/D_N3: track 91.4 -> 76.1 mm
- net /USB/D_N2: track 62.3 -> 47.4 mm
- net /USB/D_P2: track 62.3 -> 48.1 mm
- net Net-(C46-Pad1): track 0.00 -> 13.5 mm
- net /USB/D_P0: track 24.7 -> 17.7 mm
- net AVDD: track 28.4 -> 35.0 mm, vias 4 -> 3
- net /USB/D_N0: track 23.4 -> 17.3 mm
- net GND: track 106.0 -> 110.0 mm, vias 93 -> 103
- net Net-(C22-Pad1): track 8.58 -> 4.88 mm
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Other:
- board text added: "Stundner 2023 Macro Keyboard Rev. 1.0"
- board text removed: "Stundner 2023 Macro Keyboard Rev. 0.8"

Commit message: Add files via upload
Parts:
- removed U3: ~, Package_QFP:LQFP-48_7x7mm_P0.5mm
- added U9: ~, Package_SO:SSOP-28_5.3x10.2mm_P0.65mm, F.Cu at (140.7, 61.5)
- C14: footprint Capacitor_SMD:CP_Elec_4x5.8 -> Capacitor_SMD:C_0201_0603Metric_Pad0.64x0.40mm_HandSolder
- C22, C24, C26: footprint Capacitor_SMD:CP_Elec_6.3x7.7 -> Capacitor_SMD:C_1206_3216Metric_Pad1.33x1.80mm_HandSolder
- R5, R7: footprint Resistor_SMD:R_0805_2012Metric_Pad1.20x1.40mm_HandSolder -> Resistor_SMD:R_0603_1608Metric_Pad0.98x0.95mm_HandSolder
- SW1: footprint Button_Switch_THT:SW_Tactile_SPST_Angled_PTS645Vx31-2LFS -> Button_Switch_THT:SW_Tactile_SKHH_Angled
- TH1, TH2, TH4: footprint Fuse:Fuse_0805_2012Metric_Pad1.15x1.40mm_HandSolder -> Fuse:Fuse_0402_1005Metric_Pad0.77x0.64mm_HandSolder
- U5, U6, U7, U8: footprint Package_TO_SOT_SMD:TSOT-23-6 -> Package_TO_SOT_SMD:SOT-363_SC-70-6_Handsoldering
- moved D3 4.21 mm to (149.9, 57.4), turned to 180 degrees
- moved R8 2.87 mm to (150.9, 60.5), turned to 90 degrees
- moved R9 2.86 mm to (148.8, 60.5), turned to 90 degrees
- moved R5 1.82 mm to (133.5, 63.1)
- moved C26 1.57 mm to (88.9, 61.0)
- moved C22 1.14 mm to (106.9, 59.4)
Connections:
- net AVDD renamed /USB/AVDD
- net DVDD renamed /USB/DVDD
Routing:
- net /USB/D_P0: track 17.7 -> 23.3 mm
- net /USB/D_N0: track 17.3 -> 22.5 mm
- net /USB/AVDD: track 35.0 -> 39.3 mm, vias 3 -> 2
- net /USB/DVDD: track 29.1 -> 33.4 mm, vias 4 -> 0
- net /USB/D_P2: track 48.1 -> 51.6 mm
- net /USB/D_N1: track 26.3 -> 29.9 mm
- net /USB/X2: track 11.2 -> 7.87 mm
- net /USB/RESET: track 6.84 -> 10.2 mm
- net /USB/D_N2: track 47.4 -> 50.4 mm
- net /USB/D_P1: track 26.8 -> 29.6 mm
- net /USB/PGANG: track 9.67 -> 12.4 mm
- net GND: track 110.0 -> 107.6 mm, vias 103 -> 101
- net /USB/X1: track 13.3 -> 11.2 mm
- net /USB/OVERCUR1: track 10.0 -> 12.1 mm
- net +3.3V: track 60.0 -> 61.4 mm
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- removed copper zone on In2.Cu, net /USB/AVDD
- removed copper zone on In2.Cu, net /USB/DVDD

Commit message: Add files via upload
Routing:
- net +3.3V: track 61.4 -> 63.3 mm
- net /USB/D_N3: track 77.0 -> 78.7 mm
- net /USB/D_N2: track 50.4 -> 52.0 mm
- net /USB/D_N0: track 22.5 -> 23.9 mm
- net /USB/D_P3: track 77.9 -> 78.5 mm
