File: USB.kicad_sch (KiCad schematic)
At the start: 45 parts, among them J1 USB_C_Receptacle_USB2.0, J2 USB_A, J3 USB_A, J4 USB_A, U5 SRV05-4, U6 SRV05-4, Y1 12MHz

Commit message: Add files via upload
Connections:
- net D_N1: now also U5.6 (IO4); no longer U5.4 (IO3)
- net D_N2: now also U5.3 (IO2); no longer U5.1 (IO1)
- net D_N3: now also U6.6 (IO4); no longer U6.4 (IO3)
- net D_P1: now also U5.4 (IO3); no longer U5.6 (IO4)
- net D_P2: now also U5.1 (IO1); no longer U5.3 (IO2)
- net D_P3: now also U6.4 (IO3); no longer U6.6 (IO4)
- net USBD_N: now also U6.3 (IO2); no longer U6.1 (IO1)
- net USBD_P: now also U6.1 (IO1); no longer U6.3 (IO2)
Changed lines of the file:
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@@
   (junction (at 118.745 124.46) (diameter 0) (color 0 0 0 0)
   )
-  (junction (at 106.68 129.54) (diameter 0) (color 0 0 0 0)
+  (junction (at 104.775 129.54) (diameter 0) (color 0 0 0 0)
   )
   (junction (at 247.015 73.66) (diameter 0) (color 0 0 0 0)
@@
   (junction (at 43.18 170.815) (diameter 0) (color 0 0 0 0)
   )
-  (junction (at 31.75 175.895) (diameter 0) (color 0 0 0 0)
+  (junction (at 29.845 175.895) (diameter 0) (color 0 0 0 0)
   )
   (junction (at 139.065 124.46) (diameter 0) (color 0 0 0 0)
@@
   (junction (at 95.25 141.605) (diameter 0) (color 0 0 0 0)
   )
-  (junction (at 31.115 128.905) (diameter 0) (color 0 0 0 0)
-  )
-  (junction (at 105.41 132.08) (diameter 0) (color 0 0 0 0)
+  (junction (at 106.68 132.08) (diameter 0) (color 0 0 0 0)
   )
   (junction (at 252.095 73.66) (diameter 0) (color 0 0 0 0)
   )
+  (junction (at 29.845 128.905) (diameter 0) (color 0 0 0 0)
+  )
   (junction (at 257.175 66.04) (diameter 0) (color 0 0 0 0)
   )
   (junction (at 43.18 123.825) (diameter 0) (color 0 0 0 0)
   )
-  (junction (at 30.48 178.435) (diameter 0) (color 0 0 0 0)
+  (junction (at 31.115 178.435) (diameter 0) (color 0 0 0 0)
   )
   (junction (at 195.58 66.04) (diameter 0) (color 0 0 0 0)
@@
   (junction (at 267.97 116.84) (diameter 0) (color 0 0 0 0)
   )
+  (junction (at 31.75 131.445) (diameter 0) (color 0 0 0 0)
+  )
   (junction (at 63.5 123.825) (diameter 0) (color 0 0 0 0)
-  )
-  (junction (at 29.845 131.445) (diameter 0) (color 0 0 0 0)
   )
   (no_connect (at 232.41 129.54))
@@
     (stroke (width 0) (type default))
   )
+  (wire (pts (xy 31.115 168.91) (xy 53.975 168.91))
+    (stroke (width 0) (type default))
+  )
   (wire (pts (xy 144.78 154.305) (xy 144.78 156.845))
     (stroke (width 0) (type default))
   )
-  (wire (pts (xy 105.41 132.08) (xy 111.76 132.08))
+  (wire (pts (xy 106.68 132.08) (xy 111.76 132.08))
     (stroke (width 0) (type default))
   )
@@
     (stroke (width 0) (type default))
   )
+  (wire (pts (xy 31.75 131.445) (xy 31.75 139.065))
+    (stroke (width 0) (type default))
+  )
   (wire (pts (xy 139.7 154.305) (xy 144.78 154.305))
     (stroke (width 0) (type default))
   )
+  (wire (pts (xy 48.895 140.97) (xy 29.845 140.97))
+    (stroke (width 0) (type default))
+  )
   (wire (pts (xy 40.005 38.1) (xy 42.545 38.1))
     (stroke (width 0) (type default))
@@
     (stroke (width 0) (type default))
   )
-  (wire (pts (xy 31.75 168.91) (xy 53.975 168.91))
+  (wire (pts (xy 106.68 140.335) (xy 129.54 140.335))
     (stroke (width 0) (type default))
   )
@@
     (stroke (width 0) (type default))
   )
-  (wire (pts (xy 31.115 128.905) (xy 36.195 128.905))
-    (stroke (width 0) (type default))
-  )
   (wire (pts (xy 118.745 132.08) (xy 118.745 133.35))
     (stroke (width 0) (type default))
@@
     (stroke (width 0) (type default))
   )
-  (wire (pts (xy 129.54 139.7) (xy 106.68 139.7))
-    (stroke (width 0) (type default))
-  )
   (wire (pts (xy 59.055 25.4) (xy 61.595 25.4))
     (stroke (width 0) (type default))
@@
     (stroke (width 0) (type default))
   )
+  (wire (pts (xy 29.845 128.905) (xy 36.195 128.905))
+    (stroke (width 0) (type default))
+  )
   (wire (pts (xy 124.46 167.005) (xy 124.46 172.085))
     (stroke (width 0) (type default))
   )
+  (wire (pts (xy 31.75 139.065) (xy 53.975 139.065))
+    (stroke (width 0) (type default))
+  )
   (wire (pts (xy 272.415 63.5) (xy 272.415 66.04))
     (stroke (width 0) (type default))
@@
     (stroke (width 0) (type default))
   )
-  (wire (pts (xy 106.68 139.7) (xy 106.68 129.54))
-    (stroke (width 0) (type default))
-  )
-  (wire (pts (xy 30.48 178.435) (xy 36.195 178.435))
+  (wire (pts (xy 104.775 129.54) (xy 104.775 141.605))
+    (stroke (width 0) (type default))
+  )
+  (wire (pts (xy 31.115 178.435) (xy 36.195 178.435))
     (stroke (width 0) (type default))
   )
@@
     (stroke (width 0) (type default))
   )
-  (wire (pts (xy 129.54 141.605) (xy 129.54 139.7))
-    (stroke (width 0) (type default))
-  )
   (wire (pts (xy 95.25 141.605) (xy 95.25 143.51))
     (stroke (width 0) (type default))
@@
     (stroke (width 0) (type default))
   )
-  (wire (pts (xy 30.48 167.64) (xy 48.895 167.64))
-    (stroke (width 0) (type default))
-  )
-  (wire (pts (xy 31.115 139.065) (xy 31.115 128.905))
+  (wire (pts (xy 104.775 141.605) (xy 124.46 141.605))
     (stroke (width 0) (type default))
   )
@@
     (stroke (width 0) (type default))
   )
-  (wire (pts (xy 105.41 141.605) (xy 105.41 132.08))
-    (stroke (width 0) (type default))
-  )
   (wire (pts (xy 93.98 141.605) (xy 95.25 141.605))
     (stroke (width 0) (type default))
   )
+  (wire (pts (xy 29.845 168.275) (xy 48.895 168.275))
+    (stroke (width 0) (type default))
+  )
   (wire (pts (xy 252.095 73.66) (xy 257.175 73.66))
     (stroke (width 0) (type default))
@@
     (stroke (width 0) (type default))
   )
+  (wire (pts (xy 31.75 131.445) (xy 36.195 131.445))
+    (stroke (width 0) (type default))
+  )
   (wire (pts (xy 191.77 66.04) (xy 195.58 66.04))
     (stroke (width 0) (type default))
@@
     (stroke (width 0) (type default))
   )
-  (wire (pts (xy 28.575 178.435) (xy 30.48 178.435))
+  (wire (pts (xy 28.575 178.435) (xy 31.115 178.435))
     (stroke (width 0) (type default))
   )
@@
     (stroke (width 0) (type default))
   )
-  (wire (pts (xy 104.14 132.08) (xy 105.41 132.08))
+  (wire (pts (xy 104.14 132.08) (xy 106.68 132.08))
     (stroke (width 0) (type default))
   )
@@
     (stroke (width 0) (type default))
   )
-  (wire (pts (xy 124.46 141.605) (xy 105.41 141.605))
-    (stroke (width 0) (type default))
-  )
   (wire (pts (xy 232.41 116.84) (xy 247.65 116.84))
     (stroke (width 0) (type default))
@@
     (stroke (width 0) (type default))
   )
-  (wire (pts (xy 48.895 167.64) (xy 48.895 166.37))
+  (wire (pts (xy 48.895 166.37) (xy 48.895 168.275))
     (stroke (width 0) (type default))
   )
@@
     (stroke (width 0) (type default))
   )
-  (wire (pts (xy 30.48 178.435) (xy 30.48 167.64))
+  (wire (pts (xy 31.115 178.435) (xy 31.115 168.91))
     (stroke (width 0) (type default))
   )
@@
     (stroke (width 0) (type default))
   )
-  (wire (pts (xy 53.975 139.065) (xy 31.115 139.065))
-    (stroke (width 0) (type default))
-  )
   (wire (pts (xy 146.685 89.535) (xy 146.685 92.075))
     (stroke (width 0) (type default))
@@
     (stroke (width 0) (type default))
   )
-  (wire (pts (xy 29.845 140.97) (xy 29.845 131.445))
-    (stroke (width 0) (type default))
-  )
   (wire (pts (xy 63.5 123.825) (xy 71.12 123.825))
     (stroke (width 0) (type default))
   )
+  (wire (pts (xy 129.54 140.335) (xy 129.54 141.605))
+    (stroke (width 0) (type default))
+  )
   (wire (pts (xy 28.575 123.825) (xy 43.18 123.825))
     (stroke (width 0) (type default))
   )
+  (wire (pts (xy 53.975 139.065) (xy 53.975 140.97))
+    (stroke (width 0) (type default))
+  )
   (wire (pts (xy 52.705 18.415) (xy 52.705 20.32))
     (stroke (width 0) (type default))
@@
     (stroke (width 0) (type default))
   )
-  (wire (pts (xy 48.895 140.97) (xy 29.845 140.97))
-    (stroke (width 0) (type default))
-  )
   (wire (pts (xy 56.515 95.885) (xy 65.405 95.885))
     (stroke (width 0) (type default))
@@
     (stroke (width 0) (type default))
   )
-  (wire (pts (xy 53.975 140.97) (xy 53.975 139.065))
-    (stroke (width 0) (type default))
-  )
   (wire (pts (xy 201.93 109.22) (xy 207.01 109.22))
     (stroke (width 0) (type default))
@@
     (stroke (width 0) (type default))
   )
-  (wire (pts (xy 31.75 175.895) (xy 36.195 175.895))
+  (wire (pts (xy 29.845 175.895) (xy 36.195 175.895))
     (stroke (width 0) (type default))
   )
@@
     (stroke (width 0) (type default))
   )
-  (wire (pts (xy 31.75 175.895) (xy 31.75 168.91))
+  (wire (pts (xy 29.845 168.275) (xy 29.845 175.895))
     (stroke (width 0) (type default))
   )
@@
     (stroke (width 0) (type default))
   )
+  (wire (pts (xy 29.845 140.97) (xy 29.845 128.905))
+    (stroke (width 0) (type default))
+  )
   (wire (pts (xy 65.405 95.885) (xy 65.405 98.425))
     (stroke (width 0) (type default))
@@
     (stroke (width 0) (type default))
   )
-  (wire (pts (xy 106.68 129.54) (xy 111.76 129.54))
+  (wire (pts (xy 104.775 129.54) (xy 111.76 129.54))
+    (stroke (width 0) (type default))
+  )
+  (wire (pts (xy 106.68 132.08) (xy 106.68 140.335))
     (stroke (width 0) (type default))
   )
@@
     (stroke (width 0) (type default))
   )
-  (wire (pts (xy 28.575 131.445) (xy 29.845 131.445))
-    (stroke (width 0) (type default))
-  )
   (wire (pts (xy 65.405 95.885) (xy 73.025 95.885))
     (stroke (width 0) (type default))
@@
     (stroke (width 0) (type default))
   )
-  (wire (pts (xy 104.14 129.54) (xy 106.68 129.54))
-    (stroke (width 0) (type default))
-  )
-  (wire (pts (xy 29.845 131.445) (xy 36.195 131.445))
-    (stroke (width 0) (type default))
-  )
-  (wire (pts (xy 28.575 128.905) (xy 31.115 128.905))
-    (stroke (width 0) (type default))
-  )
-  (wire (pts (xy 28.575 175.895) (xy 31.75 175.895))
+  (wire (pts (xy 104.14 129.54) (xy 104.775 129.54))
+    (stroke (width 0) (type default))
+  )
+  (wire (pts (xy 28.575 131.445) (xy 31.75 131.445))
+    (stroke (width 0) (type default))
+  )
+  (wire (pts (xy 28.575 128.905) (xy 29.845 128.905))
+    (stroke (width 0) (type default))
+  )
+  (wire (pts (xy 28.575 175.895) (xy 29.845 175.895))
     (stroke (width 0) (type default))
   )
@@
     (effects (font (size 1.27 1.27)) (justify left bottom))
   )
-  (label "D_N0" (at 124.46 172.085 90) (fields_autoplaced)
+  (label "D_N0" (at 129.54 172.085 90) (fields_autoplaced)
     (effects (font (size 1.27 1.27)) (justify left bottom))
   )
@@
     (effects (font (size 1.27 1.27)) (justify left bottom))
   )
-  (label "D_P0" (at 129.54 172.085 90) (fields_autoplaced)
-    (effects (font (size 1.27 1.27)) (justify left bottom))
-  )
+  (label "D_P0" (at 124.46 172.085 90) (fields_autoplaced)
+    (effects (font (size 1.27 1.27)) (justify left bottom))
+  )

Commit message: Add files via upload
Parts:
- removed C10, C11, C13, C14, C18: 0.1uF, Capacitor_SMD:C_0805_2012Metric_Pad1.18x1.45mm_HandSolder, symbol Device:C
- removed C12: 1uF, Capacitor_SMD:CP_Elec_4x5.4, symbol Device:C
- removed C17: 10uF, Capacitor_SMD:CP_Elec_4x5.8, symbol Device:C_Polarized_US
- removed FB1: BLM18BA, Inductor_SMD:L_0603_1608Metric_Pad1.05x0.95mm_HandSolder, symbol Device:FerriteBead
- added C37, C38, C39, C40: 1uF, Capacitor_SMD:C_0603_1608Metric_Pad1.08x0.95mm_HandSolder, symbol Device:C
- added C41, C42: 0.1uF, Capacitor_SMD:C_0603_1608Metric_Pad1.08x0.95mm_HandSolder, symbol Device:C
- added FB1 (x2): BLM18BA, Inductor_SMD:L_0603_1608Metric_Pad1.05x0.95mm_HandSolder, symbol Device:FerriteBead
- C15, C19, C20, C21, C23, C27, C29: footprint Capacitor_SMD:C_0805_2012Metric_Pad1.18x1.45mm_HandSolder -> Capacitor_SMD:C_0603_1608Metric_Pad1.08x0.95mm_HandSolder
- C16: footprint Capacitor_SMD:CP_Elec_4x5.4 -> Capacitor_SMD:C_0603_1608Metric_Pad1.08x0.95mm_HandSolder
- R10, R11, R12, R13, R17, R5, R6, R7, R8, R9: footprint Resistor_SMD:R_1206_3216Metric_Pad1.30x1.75mm_HandSolder -> Resistor_SMD:R_0805_2012Metric_Pad1.20x1.40mm_HandSolder
Connections:
- net +3.3V: now also C37.1, C38.1, FB1.1, FB1.1; no longer U3.1 (AVDD), U3.12 (AVDD), U3.16 (AVDD), U3.19 (AVDD), U3.7 (AVDD)
- net AGND: now also C37.2, C38.2, C39.2, C40.2, C41.1, C42.1
- net DVDD: now also C40.1, C41.2, FB1.2
- new net AVDD: C39.1, C42.2, FB1.2, U3.1 (AVDD), U3.12 (AVDD), U3.16 (AVDD), U3.19 (AVDD), U3.7 (AVDD)
Other:
- moved on the sheet: C15, C16

Commit message: Add files via upload
Parts:
- added C10, C11, C12, C13, C17, C18, C43, C44: 0.1uF, Capacitor_SMD:C_0603_1608Metric_Pad1.08x0.95mm_HandSolder, symbol Device:C
Connections:
- net AGND: now also C10.1, C11.1, C12.1, C13.1, C17.1, C18.1, C43.1, C44.1
- net AVDD: now also C10.2, C11.2, C12.2, C13.2
- net DVDD: now also C17.2, C18.2, C43.2, C44.2
Other:
- note added: "Pro Pin am Ic 100nF"
- moved on the sheet: C37, C38, C39, C40, C41, C42, FB1

Commit message: Add files via upload
Connections:
- net D_N1: now also U5.4 (IO3); no longer U5.6 (IO4)
- net D_N2: now also U6.3 (IO2); no longer U5.3 (IO2)
- net D_P1: now also U5.6 (IO4); no longer U5.4 (IO3)
- net D_P2: now also U6.1 (IO1); no longer U5.1 (IO1)
- net USBD_N: now also U3.21 (DM4); no longer J1.A7 (D-), J1.B7 (D-), U3.3 (DM0), U6.3 (IO2)
- net USBD_P: now also U3.22 (DP4); no longer J1.A6 (D+), J1.B6 (D+), U3.4 (DP0), U6.1 (IO1)
- new net D_N0: J1.A7 (D-), J1.B7 (D-), U3.3 (DM0), U5.3 (IO2)
- new net D_P0: J1.A6 (D+), J1.B6 (D+), U3.4 (DP0), U5.1 (IO1)
- no-connect marks 9 -> 7
Other:
- moved on the sheet: C26, C27, FB1, J3, TH2

Commit message: Add files via upload
Parts:
- removed U5, U6: SRV05-4, Package_TO_SOT_SMD:SOT-23-6, symbol Power_Protection:SRV05-4
- added U5, U6, U7, U8: NUP2202, Package_TO_SOT_SMD:TSOT-23-6, symbol Power_Protection:NUP2202
Connections:
- net +5V: now also U5.5, U6.5, U7.5, U8.5
- net AGND: now also U5.2, U6.2, U7.2, U8.2
- net D_N0: now also U5.6
- net D_N1: now also U7.6
- net D_N2: now also U8.6
- net D_N3: now also U6.6
- net D_P0: now also U5.1
- net D_P1: now also U7.1
- net D_P2: now also U8.1
- net D_P3: now also U6.1
